Commit message: Added map_image_generator

File: turtlebot3_beam_description/urdf/turtlebot3_waffle.gazebo.xacro (robot description, xacro)
@@ -134,46 +134,3 @@
     </sensor>
   </gazebo>
-  <gazebo reference="bottom_camera_rgb_frame">
-    <sensor type="depth" name="realsense_R200">
-      <always_on>true</always_on>
-      <visualize>$(arg camera_visual)</visualize>
-      <camera>
-          <horizontal_fov>1.3439</horizontal_fov>
-          <image>
-              <width>1920</width>
-              <height>1080</height>
-              <format>R8G8B8</format>
-          </image>
-          <depth_camera></depth_camera>
-          <clip>
-              <near>0.03</near>
-              <far>100</far>
-          </clip>
-      </camera>
-      <plugin name="camera_controller" filename="libgazebo_ros_openni_kinect.so">
-        <baseline>0.2</baseline>
-        <alwaysOn>true</alwaysOn>
-        <updateRate>30.0</updateRate>
-        <cameraName>bottom_camera</cameraName>
-        <frameName>camera_rgb_optical_frame</frameName>
-        <imageTopicName>rgb/image_raw</imageTopicName>
-        <depthImageTopicName>depth/image_raw</depthImageTopicName>
-        <pointCloudTopicName>depth/points</pointCloudTopicName>
-        <cameraInfoTopicName>rgb/camera_info</cameraInfoTopicName>
-        <depthImageCameraInfoTopicName>depth/camera_info</depthImageCameraInfoTopicName>
-        <pointCloudCutoff>0.4</pointCloudCutoff>
-            <hackBaseline>0.07</hackBaseline>
-            <distortionK1>0.0</distortionK1>
-            <distortionK2>0.0</distortionK2>
-            <distortionK3>0.0</distortionK3>
-            <distortionT1>0.0</distortionT1>
-            <distortionT2>0.0</distortionT2>
-        <CxPrime>0.0</CxPrime>
-        <Cx>0.0</Cx>
-        <Cy>0.0</Cy>
-        <focalLength>0</focalLength>
-        <hackBaseline>0</hackBaseline>
-      </plugin>
-    </sensor>
-  </gazebo>
 </robot>

File: turtlebot3_beam_description/urdf/turtlebot3_waffle.urdf.xacro (robot description, xacro)
@@ -4,4 +4,5 @@
   <xacro:include filename="$(find turtlebot3_description)/urdf/turtlebot3_waffle.gazebo.xacro"/>
   <xacro:include filename="$(find turtlebot3_beam_description)/urdf/accessories/camera.urdf.xacro"/>
+  <xacro:include filename="$(find turtlebot3_beam_description)/urdf/accessories/r200.urdf.xacro"/>
   <xacro:property name="r200_cam_rgb_px" value="0.005"/>
   <xacro:property name="r200_cam_rgb_py" value="0.018"/>
@@ -167,9 +168,9 @@
   <!-- Front camera -->
   <xacro:camera_sensor name="front_camera" parent="base_link" hfov="1.3439" image_width="1920" image_height="1080"  >
-    <origin xyz="0.064 -0.065 1.2" rpy="0 0 0" />
+    <origin xyz="0.064 0 1.2" rpy="0 0 0" />
   </xacro:camera_sensor>
   <!-- Bottom camera -->
-  <xacro:camera_sensor name="bottom_camera" parent="base_link" hfov="1.3439" image_width="1920" image_height="1080"  >
-    <origin xyz="0.064 -0.065 1.1" rpy="0 0.523599 0" />
-  </xacro:camera_sensor>
+  <xacro:r200 name="r200" parent="base_link" >
+    <origin xyz="0.064 0 1.1" rpy="0 0.523599 0" />
+  </xacro:r200>
 </robot>

Commit message: Migrate URDF to ROS2, and cleanup unused copies of stuff from the original turtlebot3_description repo

File: turtlebot3_beam_description/urdf/turtlebot3_waffle.gazebo.xacro (robot description, xacro)
@@ -53,34 +53,36 @@
   </gazebo>
   <gazebo>
+    <plugin name="joint_states" filename="libgazebo_ros_joint_state_publisher.so">
+      <joint_name>wheel_left_joint</joint_name>
+      <joint_name>wheel_right_joint</joint_name>
+    </plugin>
     <plugin name="turtlebot3_waffle_controller" filename="libgazebo_ros_diff_drive.so">
-      <commandTopic>cmd_vel</commandTopic>
-      <odometryTopic>odom</odometryTopic>
-      <odometryFrame>odom</odometryFrame>
-      <odometrySource>world</odometrySource>
-      <publishOdomTF>true</publishOdomTF>
-      <robotBaseFrame>base_footprint</robotBaseFrame>
-      <publishWheelTF>false</publishWheelTF>
-      <publishTf>true</publishTf>
-      <publishWheelJointState>true</publishWheelJointState>
-      <legacyMode>false</legacyMode>
-      <updateRate>30</updateRate>
-      <leftJoint>wheel_left_joint</leftJoint>
-      <rightJoint>wheel_right_joint</rightJoint>
-      <wheelSeparation>0.287</wheelSeparation>
-      <wheelDiameter>0.066</wheelDiameter>
-      <wheelAcceleration>1</wheelAcceleration>
-      <wheelTorque>10</wheelTorque>
-      <rosDebugLevel>na</rosDebugLevel>
+      <command_topic>cmd_vel</command_topic>
+      <odometry_topic>odom</odometry_topic>
+      <odometry_frame>odom</odometry_frame>
+      <odometry_source>world</odometry_source>
+      <publish_odom>true</publish_odom>
+      <publish_odom_tf>true</publish_odom_tf>
+      <robot_base_frame>base_footprint</robot_base_frame>
+      <publish_wheel_tf>false</publish_wheel_tf>
+      <update_rate>30</update_rate>
+      <left_joint>wheel_left_joint</left_joint>
+      <right_joint>wheel_right_joint</right_joint>
+      <wheel_separation>0.287</wheel_separation>
+      <wheel_diameter>0.066</wheel_diameter>
+      <max_wheel_acceleration>1</max_wheel_acceleration>
+      <max_wheel_torque>10</max_wheel_torque>
     </plugin>
   </gazebo>
   <gazebo>
     <plugin name="imu_plugin" filename="libgazebo_ros_imu.so">
-      <alwaysOn>true</alwaysOn>
-      <bodyName>imu_link</bodyName>
-      <frameName>imu_link</frameName>
-      <topicName>imu</topicName>
-      <serviceName>imu_service</serviceName>
-      <gaussianNoise>0.0</gaussianNoise>
-      <updateRate>0</updateRate>
+      <always_on>true</always_on>
+      <body_name>imu_link</body_name>
+      <frame_name>imu_link</frame_name>
+      <service_name>imu_service</service_name>
+      <update_rate>0</update_rate>
+      <ros>
+        <remapping>~/out:=imu</remapping>
+      </ros>
       <imu>
         <noise>
@@ -128,7 +130,10 @@
         </noise>
       </ray>
-      <plugin name="gazebo_ros_lds_lfcd_controller" filename="libgazebo_ros_laser.so">
-        <topicName>scan</topicName>
-        <frameName>base_scan</frameName>
+      <plugin name="gazebo_ros_lds_lfcd_controller" filename="libgazebo_ros_ray_sensor.so">
+        <ros>
+          <remapping>~/out:=scan</remapping>
+        </ros>
+        <frame_name>base_scan</frame_name>
+        <output_type>sensor_msgs/LaserScan</output_type>
       </plugin>
     </sensor>

File: turtlebot3_beam_description/urdf/turtlebot3_waffle.urdf.xacro (robot description, xacro)
@@ -1,5 +1,5 @@
 <?xml version="1.0" ?>
 <robot name="turtlebot3_waffle" xmlns:xacro="http://ros.org/wiki/xacro">
-  <xacro:include filename="$(find turtlebot3_description)/urdf/common_properties.urdf"/>
+  <xacro:include filename="$(find turtlebot3_beam_description)/urdf/common_properties.urdf"/>
   <xacro:include filename="$(find turtlebot3_beam_description)/urdf/turtlebot3_waffle.gazebo.xacro"/>
   <xacro:include filename="$(find turtlebot3_beam_description)/urdf/accessories/camera.urdf.xacro"/>
@@ -19,5 +19,5 @@
       <origin xyz="-0.064 0 0.0" rpy="0 0 0"/>
       <geometry>
-        <mesh filename="package://turtlebot3_description/meshes/bases/waffle_base.stl" scale="0.001 0.001 0.001"/>
+        <mesh filename="package://turtlebot3_beam_description/meshes/bases/waffle_base.stl" scale="0.001 0.001 0.001"/>
       </geometry>
       <material name="light_black"/>
@@ -47,5 +47,5 @@
       <origin xyz="0 0 0" rpy="1.57 0 0"/>
       <geometry>
-        <mesh filename="package://turtlebot3_description/meshes/wheels/left_tire.stl" scale="0.001 0.001 0.001"/>
+        <mesh filename="package://turtlebot3_beam_description/meshes/wheels/left_tire.stl" scale="0.001 0.001 0.001"/>
       </geometry>
       <material name="dark"/>
@@ -75,5 +75,5 @@
       <origin xyz="0 0 0" rpy="1.57 0 0"/>
       <geometry>
-        <mesh filename="package://turtlebot3_description/meshes/wheels/right_tire.stl" scale="0.001 0.001 0.001"/>
+        <mesh filename="package://turtlebot3_beam_description/meshes/wheels/right_tire.stl" scale="0.001 0.001 0.001"/>
       </geometry>
       <material name="dark"/>
@@ -148,5 +148,5 @@
       <origin xyz="0 0 0" rpy="0 0 0"/>
       <geometry>
-        <mesh filename="package://turtlebot3_description/meshes/sensors/lds.stl" scale="0.001 0.001 0.001"/>
+        <mesh filename="package://turtlebot3_beam_description/meshes/sensors/lds.stl" scale="0.001 0.001 0.001"/>
       </geometry>
       <material name="dark"/>
